Commit message: Add ultrasonic sensors, sensor fusion costmap, Nav2 Ackermann config, new open maze world, smart backup recovery

File: src/limo_ros2/limo_car/gazebo/ackermann_with_sensor.xacro (robot description, xacro)
@@ -37,3 +37,24 @@
         <child link="imu_link"/>
     </joint>
+    <!-- ************************* Front Ultrasonic ******************* -->
+    <xacro:gazebo_ultrasonic_front frame_prefix="ultrasonic_front" />
+    <joint name="ultrasonic_front_joint" type="fixed">
+        <origin xyz="0.13 0.0 0.05" rpy="0 0 0"/>
+        <parent link="base_link"/>
+        <child link="ultrasonic_front_link"/>
+    </joint>
+    <!-- ************************* Left Ultrasonic ******************* -->
+    <xacro:gazebo_ultrasonic_left frame_prefix="ultrasonic_left" />
+    <joint name="ultrasonic_left_joint" type="fixed">
+        <origin xyz="0.10 0.07 0.05" rpy="0 0 0.7854"/>
+        <parent link="base_link"/>
+        <child link="ultrasonic_left_link"/>
+    </joint>
+    <!-- ************************* Right Ultrasonic ******************* -->
+    <xacro:gazebo_ultrasonic_right frame_prefix="ultrasonic_right" />
+    <joint name="ultrasonic_right_joint" type="fixed">
+        <origin xyz="0.10 -0.07 0.05" rpy="0 0 -0.7854"/>
+        <parent link="base_link"/>
+        <child link="ultrasonic_right_link"/>
+    </joint>
 </robot>

File: src/limo_ros2/limo_car/gazebo/sensor.xacro (robot description, xacro)
@@ -204,3 +204,181 @@
         </gazebo>
     </xacro:macro>
+    <!-- ************************* Front Ultrasonic ******************* -->
+    <xacro:macro name="gazebo_ultrasonic_front" params="frame_prefix">
+        <link name="${frame_prefix}_link">
+            <inertial>
+                <mass value="0.02"/>
+                <origin xyz="0 0 0" rpy="0 0 0"/>
+                <inertia ixx="1e-6" ixy="0" ixz="0"
+                         iyy="1e-6" iyz="0"
+                         izz="1e-6"/>
+            </inertial>
+            <visual>
+                <origin xyz="0 0 0" rpy="0 0 0"/>
+                <geometry>
+                    <box size="0.016 0.045 0.015"/>
+                </geometry>
+            </visual>
+            <collision>
+                <origin xyz="0 0 0" rpy="0 0 0"/>
+                <geometry>
+                    <box size="0.016 0.045 0.015"/>
+                </geometry>
+            </collision>
+        </link>
+        <gazebo reference="${frame_prefix}_link">
+            <material>Gazebo/Blue</material>
+            <sensor name="${frame_prefix}_sensor" type="ray">
+                <always_on>true</always_on>
+                <update_rate>10</update_rate>
+                <visualize>true</visualize>
+                <ray>
+                    <scan>
+                        <horizontal>
+                            <samples>5</samples>
+                            <resolution>1</resolution>
+                            <min_angle>-0.2618</min_angle>
+                            <max_angle>0.2618</max_angle>
+                        </horizontal>
+                    </scan>
+                    <range>
+                        <min>0.02</min>
+                        <max>4.0</max>
+                        <resolution>0.01</resolution>
+                    </range>
+                    <noise>
+                        <type>gaussian</type>
+                        <mean>0.0</mean>
+                        <stddev>0.005</stddev>
+                    </noise>
+                </ray>
+                <plugin name="front_ultrasonic_plugin" filename="libgazebo_ros_ray_sensor.so">
+                    <ros>
+                        <remapping>~/out:=/ultrasonic_front</remapping>
+                    </ros>
+                    <output_type>sensor_msgs/Range</output_type>
+                    <radiation_type>ultrasound</radiation_type>
+                    <frame_name>${frame_prefix}_link</frame_name>
+                </plugin>
+            </sensor>
+        </gazebo>
+    </xacro:macro>
+    <xacro:macro name="gazebo_ultrasonic_left" params="frame_prefix">
+        <link name="${frame_prefix}_link">
+            <inertial>
+                <mass value="0.02"/>
+                <origin xyz="0 0 0" rpy="0 0 0"/>
+                <inertia ixx="1e-6" ixy="0" ixz="0"
+                         iyy="1e-6" iyz="0"
+                         izz="1e-6"/>
+            </inertial>
+            <visual>
+                <origin xyz="0 0 0" rpy="0 0 0"/>
+                <geometry>
+                    <box size="0.016 0.045 0.015"/>
+                </geometry>
+            </visual>
+            <collision>
+                <origin xyz="0 0 0" rpy="0 0 0"/>
+                <geometry>
+                    <box size="0.016 0.045 0.015"/>
+                </geometry>
+            </collision>
+        </link>
+        <gazebo reference="${frame_prefix}_link">
+            <material>Gazebo/Blue</material>
+            <sensor name="${frame_prefix}_sensor" type="ray">
+                <always_on>true</always_on>
+                <update_rate>10</update_rate>
+                <visualize>true</visualize>
+                <ray>
+                    <scan>
+                        <horizontal>
+                            <samples>5</samples>
+                            <resolution>1</resolution>
+                            <min_angle>-0.2618</min_angle>
+                            <max_angle>0.2618</max_angle>
+                        </horizontal>
+                    </scan>
+                    <range>
+                        <min>0.02</min>
+                        <max>4.0</max>
+                        <resolution>0.01</resolution>
+                    </range>
+                    <noise>
+                        <type>gaussian</type>
+                        <mean>0.0</mean>
+                        <stddev>0.005</stddev>
+                    </noise>
+                </ray>
+                <plugin name="left_ultrasonic_plugin" filename="libgazebo_ros_ray_sensor.so">
+                    <ros>
+                        <remapping>~/out:=/ultrasonic_left</remapping>
+                    </ros>
+                    <output_type>sensor_msgs/Range</output_type>
+                    <radiation_type>ultrasound</radiation_type>
+                    <frame_name>${frame_prefix}_link</frame_name>
+                </plugin>
+            </sensor>
+        </gazebo>
+    </xacro:macro>
+    <xacro:macro name="gazebo_ultrasonic_right" params="frame_prefix">
+        <link name="${frame_prefix}_link">
+            <inertial>
+                <mass value="0.02"/>
+                <origin xyz="0 0 0" rpy="0 0 0"/>
+                <inertia ixx="1e-6" ixy="0" ixz="0"
+                         iyy="1e-6" iyz="0"
+                         izz="1e-6"/>
+            </inertial>
+            <visual>
+                <origin xyz="0 0 0" rpy="0 0 0"/>
+                <geometry>
+                    <box size="0.016 0.045 0.015"/>
+                </geometry>
+            </visual>
+            <collision>
+                <origin xyz="0 0 0" rpy="0 0 0"/>
+                <geometry>
+                    <box size="0.016 0.045 0.015"/>
+                </geometry>
+            </collision>
+        </link>
+        <gazebo reference="${frame_prefix}_link">
+            <material>Gazebo/Blue</material>
+            <sensor name="${frame_prefix}_sensor" type="ray">
+                <always_on>true</always_on>
+                <update_rate>10</update_rate>
+                <visualize>true</visualize>
+                <ray>
+                    <scan>
+                        <horizontal>
+                            <samples>5</samples>
+                            <resolution>1</resolution>
+                            <min_angle>-0.2618</min_angle>
+                            <max_angle>0.2618</max_angle>
+                        </horizontal>
+                    </scan>
+                    <range>
+                        <min>0.02</min>
+                        <max>4.0</max>
+                        <resolution>0.01</resolution>
+                    </range>
+                    <noise>
+                        <type>gaussian</type>
+                        <mean>0.0</mean>
+                        <stddev>0.005</stddev>
+                    </noise>
+                </ray>
+                <plugin name="right_ultrasonic_plugin" filename="libgazebo_ros_ray_sensor.so">
+                    <ros>
+                        <remapping>~/out:=/ultrasonic_right</remapping>
+                    </ros>
+                    <output_type>sensor_msgs/Range</output_type>
+                    <radiation_type>ultrasound</radiation_type>
+                    <frame_name>${frame_prefix}_link</frame_name>
+                </plugin>
+            </sensor>
+        </gazebo>
+    </xacro:macro>
 </robot>

File: src/limo_ros2/limo_car/urdf/limo_ackerman_base.xacro (robot description, xacro)
@@ -160,4 +160,14 @@
         <origin xyz="0.0 0 -0.1" rpy="0 0 0"/>
     </xacro:limo_imu>
+    <!-- Front ultrasonic sensor — mounted just ahead of the front face, centred -->
+    <xacro:limo_ultrasonic_front parent_prefix="base_link" frame_prefix="ultrasonic_front">
+    <origin xyz="0.068 0.0 -0.02" rpy="0 0 0"/>
+    </xacro:limo_ultrasonic_front>
+    <xacro:limo_ultrasonic_left parent_prefix="base_link" frame_prefix="ultrasonic_left">
+      <origin xyz="0.050 0.07 -0.02" rpy="0 0 0.7854"/>
+    </xacro:limo_ultrasonic_left>
+    <xacro:limo_ultrasonic_right parent_prefix="base_link" frame_prefix="ultrasonic_right">
+      <origin xyz="0.050 -0.07 -0.02" rpy="0 0 -0.7854"/>
+    </xacro:limo_ultrasonic_right>
     <!-- ruft Steuerscharnier mit vorderem Räder auf -->
     <xacro:limo_left_steering_hinge parent_prefix="base_link" wheel_prefix="left_steering_hinge">

File: src/limo_ros2/limo_car/urdf/limo_anteil.xacro (robot description, xacro)
@@ -164,3 +164,189 @@
         </gazebo>
     </xacro:macro>
+    <!-- FRONT ULTRASONIC SENSOR MACRO -->
+<xacro:macro name="limo_ultrasonic_front" params="parent_prefix frame_prefix *joint_pose">
+    <link name="${frame_prefix}_link">
+        <inertial>
+            <mass value="0.02"/>
+            <origin xyz="0 0 0" rpy="0 0 0"/>
+            <inertia ixx="1e-6" ixy="0" ixz="0"
+                     iyy="1e-6" iyz="0"
+                     izz="1e-6"/>
+        </inertial>
+        <visual>
+            <origin xyz="0 0 0" rpy="0 0 0"/>
+            <geometry>
+                <box size="0.016 0.045 0.015"/>
+            </geometry>
+            <material name="ultrasonic_blue">
+                <color rgba="0.1 0.1 0.8 1"/>
+            </material>
+        </visual>
+        <collision>
+            <origin xyz="0 0 0" rpy="0 0 0"/>
+            <geometry>
+                <box size="0.016 0.045 0.015"/>
+            </geometry>
+        </collision>
+    </link>
+    <joint name="${frame_prefix}_joint" type="fixed">
+        <parent link="${parent_prefix}"/>
+        <child link="${frame_prefix}_link"/>
+        <xacro:insert_block name="joint_pose"/>
+    </joint>
+    <gazebo reference="${frame_prefix}_link">
+        <material>Gazebo/Blue</material>
+        <sensor name="${frame_prefix}_sensor" type="ray">
+            <always_on>true</always_on>
+            <update_rate>10</update_rate>
+            <visualize>true</visualize>
+            <ray>
+                <scan>
+                    <horizontal>
+                        <samples>5</samples>
+                        <resolution>1</resolution>
+                        <min_angle>-0.2618</min_angle>
+                        <max_angle>0.2618</max_angle>
+                    </horizontal>
+                </scan>
+                <range>
+                    <min>0.02</min>
+                    <max>4.0</max>
+                    <resolution>0.01</resolution>
+                </range>
+                <noise>
+                    <type>gaussian</type>
+                    <mean>0.0</mean>
+                    <stddev>0.005</stddev>
+                </noise>
+            </ray>
+            <plugin name="front_ultrasonic_plugin" filename="libgazebo_ros_ray_sensor.so">
+                <ros>
+                    <remapping>~/out:=/ultrasonic_front</remapping>
+                </ros>
+                <output_type>sensor_msgs/Range</output_type>
+                <radiation_type>ultrasound</radiation_type>
+                <frame_name>ultrasonic_front_link</frame_name>
+            </plugin>
+        </sensor>
+    </gazebo>
+</xacro:macro>
+<xacro:macro name="limo_ultrasonic_left" params="parent_prefix frame_prefix *joint_pose">
+    <link name="${frame_prefix}_link">
+      <inertial>
+        <mass value="0.02"/>
+        <origin xyz="0 0 0" rpy="0 0 0"/>
+        <inertia ixx="1e-6" ixy="0" ixz="0" iyy="1e-6" iyz="0" izz="1e-6"/>
+      </inertial>
+      <visual>
+        <origin xyz="0 0 0" rpy="0 0 0"/>
+        <geometry><box size="0.016 0.045 0.015"/></geometry>
+        <material name="ultrasonic_blue"/>
+      </visual>
+      <collision>
+        <origin xyz="0 0 0" rpy="0 0 0"/>
+        <geometry><box size="0.016 0.045 0.015"/></geometry>
+      </collision>
+    </link>
+    <joint name="${frame_prefix}_joint" type="fixed">
+      <parent link="${parent_prefix}"/>
+      <child link="${frame_prefix}_link"/>
+      <xacro:insert_block name="joint_pose"/>
+    </joint>
+    <gazebo reference="${frame_prefix}_link">
+      <material>Gazebo/Blue</material>
+      <sensor name="${frame_prefix}_sensor" type="ray">
+        <always_on>true</always_on>
+        <update_rate>10</update_rate>
+        <visualize>true</visualize>
+        <ray>
+          <scan>
+            <horizontal>
+              <samples>5</samples>
+              <resolution>1</resolution>
+              <min_angle>-0.2618</min_angle>
+              <max_angle>0.2618</max_angle>
+            </horizontal>
+          </scan>
+          <range>
+            <min>0.02</min>
+            <max>4.0</max>
+            <resolution>0.01</resolution>
+          </range>
+          <noise>
+            <type>gaussian</type>
+            <mean>0.0</mean>
+            <stddev>0.005</stddev>
+          </noise>
+        </ray>
+        <plugin name="left_ultrasonic_plugin" filename="libgazebo_ros_ray_sensor.so">
+          <ros>
+            <remapping>~/out:=/ultrasonic_left</remapping>
+          </ros>
+          <output_type>sensor_msgs/Range</output_type>
+          <radiation_type>ultrasound</radiation_type>
+          <frame_name>ultrasonic_left_link</frame_name>
+        </plugin>
+      </sensor>
+    </gazebo>
+  </xacro:macro>
+  <xacro:macro name="limo_ultrasonic_right" params="parent_prefix frame_prefix *joint_pose">
+    <link name="${frame_prefix}_link">
+      <inertial>
+        <mass value="0.02"/>
+        <origin xyz="0 0 0" rpy="0 0 0"/>
+        <inertia ixx="1e-6" ixy="0" ixz="0" iyy="1e-6" iyz="0" izz="1e-6"/>
+      </inertial>
+      <visual>
+        <origin xyz="0 0 0" rpy="0 0 0"/>
+        <geometry><box size="0.016 0.045 0.015"/></geometry>
+        <material name="ultrasonic_blue"/>
+      </visual>
+      <collision>
+        <origin xyz="0 0 0" rpy="0 0 0"/>
+        <geometry><box size="0.016 0.045 0.015"/></geometry>
+      </collision>
+    </link>
+    <joint name="${frame_prefix}_joint" type="fixed">
+      <parent link="${parent_prefix}"/>
+      <child link="${frame_prefix}_link"/>
+      <xacro:insert_block name="joint_pose"/>
+    </joint>
+    <gazebo reference="${frame_prefix}_link">
+      <material>Gazebo/Blue</material>
+      <sensor name="${frame_prefix}_sensor" type="ray">
+        <always_on>true</always_on>
+        <update_rate>10</update_rate>
+        <visualize>true</visualize>
+        <ray>
+          <scan>
+            <horizontal>
+              <samples>5</samples>
+              <resolution>1</resolution>
+              <min_angle>-0.2618</min_angle>
+              <max_angle>0.2618</max_angle>
+            </horizontal>
+          </scan>
+          <range>
+            <min>0.02</min>
+            <max>4.0</max>
+            <resolution>0.01</resolution>
+          </range>
+          <noise>
+            <type>gaussian</type>
+            <mean>0.0</mean>
+            <stddev>0.005</stddev>
+          </noise>
+        </ray>
+        <plugin name="right_ultrasonic_plugin" filename="libgazebo_ros_ray_sensor.so">
+          <ros>
+            <remapping>~/out:=/ultrasonic_right</remapping>
+          </ros>
+          <output_type>sensor_msgs/Range</output_type>
+          <radiation_type>ultrasound</radiation_type>
+          <frame_name>ultrasonic_right_link</frame_name>
+        </plugin>
+      </sensor>
+    </gazebo>
+  </xacro:macro>
 </robot>
